File: 05_Lötübungsplatine/Lötübungsplatine/Lötübungsplatine.sch (KiCad schematic (older format))
At the start: 37 parts

Commit message: done 05 layout
Parts:
- removed R?: 100R, symbol Device:R
- added D1, D2, D3, D4, D5, D6, D7: LED, LED_SMD:LED_0805_2012Metric, symbol Device:LED
- added SW1: SW_Push, Button_Switch_THT:SW_PUSH_6mm, symbol Switch:SW_Push
- added TP1: GND_TP, TestPoint:TestPoint_Pad_3.0x3.0mm, symbol Connector:TestPoint
- added TP2: VCC_TP, TestPoint:TestPoint_Pad_3.0x3.0mm, symbol Connector:TestPoint
- 100n1: renamed from C?; footprint (none) -> Capacitor_SMD:C_0805_2012Metric
- J1: renamed from J?; footprint (none) -> Connector_USB:USB_Micro-B_Molex-105017-0001
- R1, R2, R3, R4, R5: renamed from R?; footprint (none) -> Resistor_SMD:R_2512_6332Metric
- R10, R6, R7, R8, R9: renamed from R?; footprint (none) -> Resistor_SMD:R_1206_3216Metric
- R11, R12, R13, R14, R15: renamed from R?; footprint (none) -> Resistor_SMD:R_0805_2012Metric
- R16, R17, R18, R19, R20: renamed from R?; footprint (none) -> Resistor_SMD:R_0603_1608Metric
- R21, R22, R23, R24, R25: renamed from R?; footprint (none) -> Resistor_SMD:R_0402_1005Metric
- R26, R27, R28, R29, R30: renamed from R?; footprint (none) -> Resistor_SMD:R_0201_0603Metric
- R31, R32, R33, R34: renamed from R?; footprint (none) -> Resistor_THT:R_Axial_DIN0204_L3.6mm_D1.6mm_P7.62mm_Horizontal
Connections:
- net labels added: GND, VCC
- wire segments 9 -> 73
- no-connect marks 0 -> 3
Other:
- moved on the sheet: 100n1
