File: 01_Tannenbaum/Tannenbaum/Tannenbaum.sch (KiCad schematic (older format))
At the start: 26 parts

Commit message: review 01 schematic
Parts:
- C?: value C -> 100n
- C?: value CP1 -> 7,4µ
Changed lines of the file:
@@
 P 4350 3400
 F 0 "C?" H 4465 3446 50  0000 L CNN
-F 1 "C" H 4465 3355 50  0000 L CNN
+F 1 "100n" H 4465 3355 50  0000 L CNN
 F 2 "" H 4388 3250 50  0001 C CNN
 F 3 "~" H 4350 3400 50  0001 C CNN
@@
 P 5000 2300
 F 0 "C?" H 5115 2346 50  0000 L CNN
-F 1 "CP1" H 5115 2255 50  0000 L CNN
+F 1 "7,4µ" H 5115 2255 50  0000 L CNN
 F 2 "" H 5000 2300 50  0001 C CNN
 F 3 "~" H 5000 2300 50  0001 C CNN

Commit message: created pcb for 01; good night
Parts:
- removed SW?: SW_Push_SPDT, symbol Switch:SW_Push_SPDT
- added SW1: SW_DPDT_x2, custom:switch_dpdt, symbol Switch:SW_DPDT_x2
- C1: renamed from C?; footprint (none) -> Capacitor_THT:C_Axial_L3.8mm_D2.6mm_P7.50mm_Horizontal
- C2: renamed from C?; footprint (none) -> Capacitor_THT:CP_Radial_D5.0mm_P2.00mm
- D10, D11, D12, D13, D2, D3, D4, D5, D6, D7, D8, D9: renamed from D?; footprint (none) -> LED_THT:LED_D5.0mm
- J1: renamed from J?; footprint (none) -> TerminalBlock:TerminalBlock_bornier-2_P5.08mm
- R1, R2, R3, R4, R5, R6, R7, R8: renamed from R?; footprint (none) -> Resistor_THT:R_Axial_DIN0204_L3.6mm_D1.6mm_P7.62mm_Horizontal
- U1: renamed from U?; footprint Package_SO:SOIC-8_3.9x4.9mm_P1.27mm -> Package_DIP:DIP-8_W7.62mm_LongPads
- gave numbers to parts that had none: 1
Connections:
- net +5V: now also D10.2 (A), D2.2 (A), D6.2 (A), SW1.1 (A); no longer R3.2, R5.2, R7.2
- net GND: now also D13.1 (K), D5.1 (K), D9.1 (K); no longer R4.1, R6.1, R8.1
- net at J1.2 (Pin_2): now also SW1.2 (B)
- net at D2.1 (K): now also R3.2; no longer D3.2 (A)
- net at R3.1: now also D3.2 (A); no longer D2.2 (A)
- net at D6.1 (K): now also R5.2; no longer D7.2 (A)
- net at R5.1: now also D7.2 (A); no longer D6.2 (A)
- net at D10.1 (K): now also R7.2; no longer D11.2 (A)
- net at R7.1: now also D11.2 (A); no longer D10.2 (A)
- net at D4.1 (K): now also R4.2; no longer D5.2 (A)
- net at D8.1 (K): now also R6.2; no longer D9.2 (A)
- net at D12.1 (K): now also R8.2; no longer D13.2 (A)
- new net: D5.2 (A), R4.1
- new net: D9.2 (A), R6.1
- new net: D13.2 (A), R8.1
- no-connect marks 2 -> 5
Other:
- moved on the sheet: D10, D13, D2, D5, D6, D9, R3, R4, R5, R6, R7, R8
