File: 01_Tannenbaum/Tannenbaum/Tannenbaum.kicad_pcb (KiCad board)
At the start: 2 copper layers, 50 x 80 mm, 26 parts, among them J1 Conn_01x02, SW1 SW_DPDT_x2, U1 NE555D

Commit message: review
Routing:
- net Net-(C2-Pad1): track 84.8 -> 87.2 mm
Other:
- board text added: "GND"
- board text added: "JANUS 2021"
- board text added: "VCC"
